Commit message: Add slam launch

File: urdf/robot_model.urdf (robot description, URDF)
Before this commit: robot diff_drive_robot, 8 links, 7 joints
Links:
- removed link lidar_link
- added link laser, mass 0.15; collision cylinder length=0.05 radius=0.05; visual cylinder length=0.05 radius=0.05
- added link livox_frame
- added link velodyne
Joints:
- added joint livox_joint: type fixed, parent laser, child livox_frame, origin xyz=0.0 0.0 0.0 rpy=0.0 0.0 0.0
- added joint velodyne_joint: type fixed, parent laser, child velodyne, origin xyz=0.0 0.0 0.0 rpy=0.0 0.0 0.0
- joint lidar_joint: child lidar_link -> laser

Commit message: Fix tf,odom,vel,pos

File: urdf/robot_model.urdf (robot description, URDF)
Before this commit: robot diff_drive_robot, 10 links, 9 joints
Joints:
- joint wheel_left_joint: origin xyz=0 -0.225 0 rpy=1.57 0 0 -> xyz=0 0.225 0 rpy=1.57 0 0
- joint wheel_right_joint: origin xyz=0 0.225 0 rpy=1.57 0 0 -> xyz=0 -0.225 0 rpy=1.57 0 0

Commit message: Update URDF

File: urdf/robot_model.urdf (robot description, URDF)
Before this commit: robot diff_drive_robot, 10 links, 9 joints
Links:
- removed link body
- added link frame, mass 1.0; collision cylinder length=0.15 radius=0.2; visual cylinder length=0.15 radius=0.2
Joints:
- joint base_joint: child body -> frame
- joint caster_backward_joint: parent body -> frame
- joint caster_forward_joint: parent body -> frame
- joint lidar_base_joint: parent body -> frame
- joint lidar_joint: parent body -> frame
- joint wheel_left_joint: parent body -> frame
- joint wheel_right_joint: parent body -> frame

Commit message: Fix param

File: urdf/robot_model.urdf (robot description, URDF)
Before this commit: robot diff_drive_robot, 10 links, 9 joints
Joints:
- joint lidar_joint: origin xyz=0.0 0.0 0.2 rpy=0 0 0 -> xyz=0.0 0.0 1.25 rpy=0 0 0

Commit message: Update URDF

File: urdf/robot_model.urdf (robot description, URDF)
Before this commit: robot diff_drive_robot, 10 links, 9 joints
Links:
- removed link velodyne
- added link imu_link
- link lidar_base: geometry collision box size=0.1 0.1 0.1; visual box size=0.1 0.1 1.0
Joints:
- removed joint velodyne_joint
- added joint imu_joint: type fixed, parent laser, child imu_link, origin xyz=0.0 0.1 0.0 rpy=0.0 3.14 0.0
- joint lidar_base_joint: origin xyz=0.0 0.0 0.125 rpy=0 0 0 -> xyz=0.0 0.0 0.5 rpy=0 0 0
- joint lidar_joint: origin xyz=0.0 0.0 1.25 rpy=0 0 0 -> xyz=0.0 0.0 1.0 rpy=0 0 0
- joint livox_joint: origin xyz=0.0 0.0 0.0 rpy=0.0 0.0 0.0 -> xyz=0.0 0.0 0.0 rpy=0.0 0.6108 0.0

Commit message: Add line link to urdf

File: urdf/robot_model.urdf (robot description, URDF)
Before this commit: robot diff_drive_robot, 10 links, 9 joints
Links:
- added link line_link
Joints:
- added joint line_joint: type fixed, parent base_link, child line_link, origin xyz=0.0 0.0 0.1 rpy=0.0  0.0 -1.57

Commit message: Add pcl_link and pcl_joint to robot_model.urdf

File: urdf/robot_model.urdf (robot description, URDF)
Before this commit: robot diff_drive_robot, 11 links, 10 joints
Links:
- added link pcl_link
Joints:
- added joint pcl_joint: type fixed, parent base_link, child pcl_link, origin xyz=0.0 0.0 0.0 rpy=0.0  0.0 -3.14

Commit message: Update RViz configuration and URDF model

File: urdf/robot_model.urdf (robot description, URDF)
Before this commit: robot diff_drive_robot, 12 links, 11 joints
Links:
- removed link line_link
Joints:
- removed joint line_joint
- joint pcl_joint: origin xyz=0.0 0.0 0.0 rpy=0.0  0.0 -3.14 -> xyz=0.0 0.0 0.0 rpy=0.0  0.0 4.712
